File: bevi.kicad_pcb (KiCad board)
At the start: 2 copper layers, 361.3 x 97.6 mm, 165 parts, among them J1 USB_B, J2 Conn_01x04, SW1 SW_PUSH, U1 ProMicro

Commit message: Update diodes position
Parts:
- moved D24 19.0 mm to (182.7, 57.9)
- moved D34 16.5 mm to (237.3, 57.9)
- moved D33 2.59 mm to (180.1, 57.9)
Routing:
- net Net-(D24-Pad2): track 4.43 -> 24.7 mm
- net Net-(D34-Pad2): track 4.43 -> 12.2 mm
- net Net-(D33-Pad2): track 4.43 -> 8.04 mm
- net row2: track 288.4 -> 291.7 mm, vias 0 -> 1

Commit message: Move diodes
Parts:
- moved D93 11.7 mm to (29.1, 112.5), turned to 0 degrees
- moved D84 11.2 mm to (29.1, 74.4), turned to 0 degrees
Routing:
- net row8: track 525.3 -> 543.2 mm
- net row9: track 583.5 -> 587.8 mm
- net Net-(D93-Pad2): track 12.8 -> 11.6 mm
- net Net-(D84-Pad2): track 12.4 -> 11.8 mm

Commit message: Update Diode Layout
Parts:
- moved D24 54.6 mm to (237.3, 57.9)
- moved D85 19.1 mm to (344.5, 39.0), turned to 270 degrees
- moved D33 16.5 mm to (163.6, 57.9)
- moved D25 16.4 mm to (256.2, 57.9)
- moved D23 2.57 mm to (161.1, 57.9)
- moved D34 2.53 mm to (239.8, 57.9)
- moved D97 2.46 mm to (342.1, 38.9)
Routing:
- net row8: track 543.2 -> 566.1 mm, vias 2 -> 3
- net Net-(D33-Pad2): track 8.04 -> 24.8 mm
- net Net-(D85-Pad2): track 15.7 -> 29.3 mm
- net Net-(D24-Pad2): track 24.7 -> 32.6 mm
- net Net-(D25-Pad2): track 4.43 -> 12.1 mm
- net Net-(D23-Pad2): track 4.43 -> 8.00 mm
- net Net-(D97-Pad2): track 14.0 -> 17.4 mm
- net Net-(D34-Pad2): track 12.2 -> 15.6 mm
- net row9: track 587.8 -> 590.1 mm
- net row2: track 291.7 -> 289.9 mm
- net row3: track 305.6 -> 304.3 mm
